Commit message: urdf

File: src/robot_bringup/urdf/argo_mini.urdf.xacro (robot description, xacro)
@@ -48,6 +48,9 @@
   <xacro:wheel side="left"  y_offset="${wheel_base/2}"/>
   <xacro:wheel side="right" y_offset="${-wheel_base/2}"/>
-  <!-- RPLidar A1 - mounted rotated 180 deg (yaw=pi), confirmed empirically -->
-  <!-- against real scan alignment. Update x/y/z if you remeasure the mount. -->
+  <!-- RPLidar A1 - facing forward, same direction as base_link +x.
+       Previously set to 180 deg; changed after confirming physical mount
+       faces forward. If scans still appear reversed, revert rpy to "0 0 3.14159" -
+       RPLidar A1's internal 0-degree scan reference sits opposite the connector,
+       which can make it appear reversed even when the housing faces forward. -->
   <link name="laser">
     <visual>
@@ -59,5 +62,5 @@
     <parent link="base_link"/>
     <child link="laser"/>
-    <origin xyz="0 0 0.1" rpy="0 0 3.14159"/>
+    <origin xyz="0 0 0.1" rpy="0 0 0"/>
   </joint>
   <!-- IMU - not populated by the current argo_mini.ino firmware (no MPU6050
